File: pcb/dimmer.sch (EAGLE design)
At the start: 56 parts, among them IC2 MAX3232CSE, U1 ATMEGA48-20AU

Commit message: modified
Parts:
- removed C7: (no value), rcl:C-EUC1206
- removed D1: BZX84CSMD, diode:BZX84CSMD
- removed LED1, LED3, LED4, LED5, LED6: (no value), led:LEDSML1206
- removed N$39, TP1, TP10, TP11, TP12, TP13, TP14, TP15, TP16, TP17, TP18, TP2, TP3, TP4, TP5, TP6, TP7, TP9: TPSQTP15SQ, testpad:TPSQTP15SQ
- removed R10, R11, R12, R13, R14, R15, R16, R4, R5, R8, R9: (no value), rcl:R-EU_R1206
- removed S1: 219-07, switch-dil:219-07
- removed U$1: P82B715, i2c:P82B715
- removed U$3: RJ45SMD, con-tycoelectronics:RJ45SMD
- removed U$6: PINHD-1X2SMD, pinhead:PINHD-1X2SMD
- added JP1: (no value), pinhead:PINHD-2X3
- added Q1: IRFR5305, transistor-power:IRFR5305
- added Q3: BC817-16LT1SMD, transistor-npn:BC817-16LT1SMD
- added X1, X4: (no value), con-wago-508:W237-02P
- added X2, X3: (no value), con-wago-508:W237-3E
- C1: device rcl:C-EUC0603 -> rcl:C-EUC1206
- C5: device rcl:C-EUC1206 -> rcl:C-EUC0603
- R2: value (none) -> 470
- R6: value (none) -> 10k
- R7: value (none) -> 1K
- U$4: value (none) -> MOC3040SMD; device pinhead:PINHD-1X3SMD -> optocoupler:MOC3040SMD
- U$5: value PINHD-1X1SMD -> BT137S; device pinhead:PINHD-1X1SMD -> triac:BT137S
- U1: value ATMEGA48-20AU -> ATTINY2313; device atmega48:ATMEGA48-20AU -> Atmel.By.element14:ATTINY2313-20SU
Connections:
- removed net +12V: R14.1, U$1.VCC, U$2.7, U$2.8
- removed net N$25 (its old number): C2.1, IC2G$1.C2+
- removed net N$29: U$4.1, U1.PB5
- removed net N$30: U$4.2, U1.PB4
- removed net N$31: U$4.3, U1.PB3
- removed net N$32: R15.1, U$5.1, U1.PC6
- removed net N$33: LED1.C, R16.1
- removed net N$34: C6.2, U1.AVCC
- removed net N$35: LED1.A, U1.PD4
- removed net N$36: C7.1, U1.AREF
- removed net N$37: LED3.A, LED4.C
- removed net N$38: LED5.C, LED6.A
- removed net N$8 (its old number): R3.2, S1.12, U1.PD5
- removed net VCC: TP3.TP, TP4.TP
- new net VCC+12V: C6.1, R7.1, U$2.7, X1-1.KL, X4-2.KL
- new net VCC+5V: C1.1, C5.2, JP1.2, R3.1, U$2.5, U1.VCC
- net GND: now also C1.2, C6.2, JP1.6, Q1.S, Q3.E, U$2.2, U$2.4, U$2.8, U$4.C, X1-2.KL; no longer C5.2, C7.2, D1.A, LED3.C, LED6.C, R10.2, R11.2, R12.2, R13.2, R16.2, R8.2, R9.2, S1.1, S1.2, S1.3, S1.4, S1.5, S1.6, S1.7, TP11.TP, TP13.TP, TP15.TP, TP16.TP, TP17.TP, TP18.TP, TP2.TP, U$1.GND, U$2.5, U$3.5, U$3.6, U$6.2, U1.GND_2, U1.GND_3
- net N$1: now also R2.2, U$5.G; no longer U$1.SCL, U1.PC5
- net N$12: now also Q1.G, Q3.C, R7.2; no longer U$1.LDA, U$2.1, U$2.2
- net N$13: now also R6.1, U1.PB2; no longer U$1.LCL, U$2.3, U$2.4
- net N$14: now also R1.2, U1.PB3; no longer R12.1, TP14.TP, U1.ADC6
- net N$15: now also Q1.D, X4-1.KL; no longer R11.1, TP10.TP, U1.ADC7
- net N$16: now also X2-1.KL, X3-3.KL; no longer N$39.TP, R10.1, U1.PC0
- net N$17: now also X2-2.KL, X3-2.KL; no longer R9.1, TP12.TP, U1.PC1
- net N$18: now also U$5.A1, X3-1.KL; no longer R8.1, TP9.TP, U1.PC2
- net N$19: now also U$4.A2, U$5.A2, X2-3.KL; no longer R13.1, TP7.TP, U1.PC3
- net N$2: now also Q3.B, R6.2; no longer U$1.SDA, U1.PC4
- net N$20: now also R2.1, U$4.A1; no longer C1.1, IC2G$1.C1+
- net N$21: now also IC2G$1.C2-; no longer C5.1, C6.1, D1.C, LED4.A, LED5.A, R1.1, R14.2, R15.2, R2.1, R3.1, R4.1, R5.1, R6.1, R7.1, TP5.TP, TP6.TP, U$3.7, U$3.8, U$6.1, U1.VCC, U1.VCC_2
- net N$22: now also C3.2, IC2G$1.C2+; no longer C1.2, IC2G$1.C1-
- net N$23: now also C2.1, IC2G$1.C1-; no longer IC2G$1.T1OUT, U$3.1, U$3.2
- net N$24: now also C2.2, IC2G$1.C1+; no longer IC2G$1.R1IN, U$3.3, U$3.4
- net N$26: now also C5.1, IC2G$1.V+; no longer C2.2, IC2G$1.C2-
- net N$27: now also JP1.5, R3.2, U1.PA2; no longer C3.2, IC2G$1.V+
- net N$3: now also IC2G$1.R1IN, U$2.1; no longer R1.2, S1.14, U1.PB6
- net N$4: now also IC2G$1.T1OUT, U$2.3; no longer R7.2, S1.8, U1.PB1
- net N$5: now also JP1.3, U1.PB7; no longer R6.2, S1.9, U1.PB0
- net N$6: now also JP1.1, U1.PB6; no longer R5.2, S1.10, U1.PD7
- net N$7: now also JP1.4, U1.PB5; no longer R4.2, S1.11, U1.PD6
- net N$9: now also R1.1, U$4.A; no longer R2.2, S1.13, U1.PB7
Other:
- moved on the sheet: C1, C2, C3, C4, C5, C6, IC2, R1, R2, R3, R6, R7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

Commit message: sleep mode
Connections:
- net GND: now also U$2.5; no longer U$2.2, U$2.4, U$2.8
- net N$3: now also U$2.2
- net N$4: now also U$2.4
- net VCC+12V: no longer U$2.7
- net VCC+5V: now also U$2.7, U$2.8; no longer U$2.5
Other:
- moved on the sheet: U$2
Changed lines of the file:
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@@
 <setting verticaltext="up"/>
 </settings>
-<grid distance="6.25" unitdist="mil" unit="mil" style="lines" multiple="1" display="no" altdistance="0.01" altunitdist="inch" altunit="inch"/>
+<grid distance="0.025" unitdist="inch" unit="inch" style="lines" multiple="1" display="no" altdistance="0.01" altunitdist="inch" altunit="inch"/>
 <layers>
 <layer number="1" name="Top" color="4" fill="1" visible="no" active="no"/>
@@
 <part name="U$4" library="optocoupler" deviceset="MOC3040SMD" device=""/>
 <part name="GND1" library="supply1" deviceset="GND" device=""/>
-<part name="GND2" library="supply1" deviceset="GND" device=""/>
 <part name="GND3" library="supply1" deviceset="GND" device=""/>
 <part name="GND4" library="supply1" deviceset="GND" device=""/>
@@
 <part name="SUPPLY5" library="supply2" deviceset="VCC" device="" value="5V"/>
 <part name="Q3" library="transistor-npn" deviceset="BC817*" device="SMD" technology="-16LT1"/>
+<part name="GND2" library="supply1" deviceset="GND" device=""/>
 </parts>
 <sheets>
@@
 <instance part="Q1" gate="G$1" x="69.215" y="32.0675" rot="MR180"/>
 <instance part="R1" gate="G$1" x="52.07" y="64.77" rot="R180"/>
-<instance part="U$2" gate="G$1" x="-69.85" y="87.63" rot="MR0"/>
+<instance part="U$2" gate="G$1" x="-73.66" y="87.63" rot="MR0"/>
 <instance part="X2" gate="-1" x="114.6175" y="14.605" rot="R180"/>
 <instance part="X2" gate="-2" x="113.9825" y="20.6375" rot="R180"/>
@@
 <instance part="U$4" gate="G$1" x="70.1675" y="59.69"/>
 <instance part="GND1" gate="1" x="57.15" y="13.97"/>
-<instance part="GND2" gate="1" x="-63.1825" y="57.785"/>
 <instance part="GND3" gate="1" x="-49.37125" y="57.785"/>
 <instance part="GND4" gate="1" x="5.3975" y="67.31"/>
 <instance part="GND5" gate="1" x="83.34375" y="87.63"/>
-<instance part="SUPPLY1" gate="G$1" x="-42.38625" y="85.09" smashed="yes" rot="R270">
-<attribute name="VALUE" x="-38.57625" y="84.1375" size="1.778" layer="96"/>
+<instance part="SUPPLY1" gate="G$1" x="-71.12" y="60.16625" smashed="yes" rot="R180">
+<attribute name="VALUE" x="-72.0725" y="56.35625" size="1.778" layer="96" rot="R270"/>
 </instance>
 <instance part="GND" gate="1" x="-42.545" y="57.785"/>
@@
 <attribute name="VALUE" x="3.4925" y="109.37875" size="1.778" layer="96"/>
 </instance>
-<instance part="VCC+12V" gate="G$1" x="-42.38625" y="80.01" smashed="yes" rot="R270">
-<attribute name="VALUE" x="-38.89375" y="79.375" size="1.778" layer="96"/>
+<instance part="VCC+12V" gate="G$1" x="-13.81125" y="57.785" smashed="yes" rot="R270">
+<attribute name="VALUE" x="-10.31875" y="57.15" size="1.778" layer="96"/>
 </instance>
 <instance part="VCC+12V1" gate="G$1" x="61.2775" y="44.1325" smashed="yes" rot="R90">
@@
 </instance>
 <instance part="Q3" gate="G$1" x="61.2775" y="24.4475"/>
+<instance part="GND2" gate="1" x="-63.5" y="57.785"/>
 </instances>
 <busses>
@@
 </net>
 <net name="GND" class="0">
-<segment>
-<wire x1="-63.1825" y1="77.47" x2="-63.1825" y2="82.55" width="0.1524" layer="91"/>
-<wire x1="-63.1825" y1="82.55" x2="-63.1825" y2="87.63" width="0.1524" layer="91"/>
-<wire x1="-63.1825" y1="92.71" x2="-63.1825" y2="87.63" width="0.1524" layer="91"/>
-<wire x1="-63.1825" y1="77.47" x2="-63.1825" y2="60.325" width="0.1524" layer="91"/>
-<junction x="-63.1825" y="87.63"/>
-<junction x="-63.1825" y="82.55"/>
-<junction x="-63.1825" y="77.47"/>
-<pinref part="GND2" gate="1" pin="GND"/>
-<wire x1="-63.1825" y1="92.71" x2="-67.31" y2="92.71" width="0.1524" layer="91"/>
-<wire x1="-63.1825" y1="87.63" x2="-67.31" y2="87.63" width="0.1524" layer="91"/>
-<wire x1="-63.1825" y1="82.55" x2="-67.31" y2="82.55" width="0.1524" layer="91"/>
-<wire x1="-67.31" y1="77.47" x2="-63.1825" y2="77.47" width="0.1524" layer="91"/>
-<pinref part="U$2" gate="G$1" pin="4"/>
-<pinref part="U$2" gate="G$1" pin="6"/>
-<pinref part="U$2" gate="G$1" pin="8"/>
-<pinref part="U$2" gate="G$1" pin="2"/>
-</segment>
 <segment>
 <pinref part="U1" gate="A" pin="GND"/>
@@
 <wire x1="-56.35625" y1="60.325" x2="-56.35625" y2="62.23" width="0.1524" layer="91"/>
 </segment>
+<segment>
+<pinref part="U$2" gate="G$1" pin="5"/>
+<pinref part="U$2" gate="G$1" pin="6"/>
+<wire x1="-71.12" y1="85.09" x2="-71.12" y2="82.55" width="0.1524" layer="91"/>
+<wire x1="-71.12" y1="82.55" x2="-63.5" y2="82.55" width="0.1524" layer="91"/>
+<wire x1="-63.5" y1="82.55" x2="-63.5" y2="60.325" width="0.1524" layer="91"/>
+<pinref part="GND2" gate="1" pin="GND"/>
+<junction x="-71.12" y="82.55"/>
+</segment>
 </net>
 <net name="N$8" class="0">
@@
 <segment>
 <pinref part="C1" gate="G$1" pin="1"/>
-<wire x1="-49.37125" y1="85.09" x2="-44.92625" y2="85.09" width="0.1524" layer="91"/>
 <wire x1="-49.37125" y1="69.85" x2="-49.37125" y2="85.09" width="0.1524" layer="91"/>
-<junction x="-49.37125" y="85.09"/>
-<pinref part="SUPPLY1" gate="G$1" pin="VCC"/>
-<wire x1="-49.37125" y1="85.09" x2="-67.31" y2="85.09" width="0.1524" layer="91"/>
-<pinref part="U$2" gate="G$1" pin="5"/>
 </segment>
 <segment>
@@
 <pinref part="R3" gate="G$1" pin="1"/>
 <pinref part="SUPPLY5" gate="G$1" pin="VCC"/>
+</segment>
+<segment>
+<pinref part="U$2" gate="G$1" pin="7"/>
+<pinref part="U$2" gate="G$1" pin="8"/>
+<wire x1="-71.12" y1="77.47" x2="-71.12" y2="80.01" width="0.1524" layer="91"/>
+<wire x1="-71.12" y1="77.47" x2="-71.12" y2="62.70625" width="0.1524" layer="91"/>
+<pinref part="SUPPLY1" gate="G$1" pin="VCC"/>
+<wire x1="-71.12" y1="62.70625" x2="-70.485" y2="62.865" width="0.1524" layer="91"/>
+<junction x="-71.12" y="62.70625"/>
+<junction x="-71.12" y="77.47"/>
 </segment>
 </net>
@@
 <pinref part="U$2" gate="G$1" pin="1"/>
 <pinref part="IC2" gate="G$1" pin="R1IN"/>
-<wire x1="-67.31" y1="95.25" x2="-35.56" y2="95.25" width="0.1524" layer="91"/>
+<wire x1="-71.12" y1="95.25" x2="-35.56" y2="95.25" width="0.1524" layer="91"/>
+<pinref part="U$2" gate="G$1" pin="2"/>
+<wire x1="-71.12" y1="92.71" x2="-71.12" y2="95.25" width="0.1524" layer="91"/>
+<junction x="-71.12" y="95.25"/>
 </segment>
 </net>
@@
 <pinref part="U$2" gate="G$1" pin="3"/>
 <pinref part="IC2" gate="G$1" pin="T1OUT"/>
-<wire x1="-67.31" y1="90.17" x2="-35.56" y2="90.17" width="0.1524" layer="91"/>
+<wire x1="-71.12" y1="90.17" x2="-35.56" y2="90.17" width="0.1524" layer="91"/>
+<pinref part="U$2" gate="G$1" pin="4"/>
+<wire x1="-71.12" y1="87.63" x2="-71.12" y2="90.17" width="0.1524" layer="91"/>
+<junction x="-71.12" y="90.17"/>
 </segment>
 </net>
@@
 <net name="VCC+12V" class="0">
 <segment>
-<pinref part="VCC+12V" gate="G$1" pin="VCC"/>
-<wire x1="-67.31" y1="80.01" x2="-56.35625" y2="80.01" width="0.1524" layer="91"/>
-<pinref part="U$2" gate="G$1" pin="7"/>
 <pinref part="C6" gate="G$1" pin="1"/>
-<wire x1="-56.35625" y1="80.01" x2="-44.92625" y2="80.01" width="0.1524" layer="91"/>
 <wire x1="-56.35625" y1="69.85" x2="-56.35625" y2="80.01" width="0.1524" layer="91"/>
-<junction x="-56.35625" y="80.01"/>
-</segment>
-<segment>
+</segment>
+<segment>
