File: pcb/dimmer.v2.sch (EAGLE design)
At the start: 45 parts, among them M328 ATMEGA328P-AU, SW1 RJ45SMD, SW2 RJ45SMD, SW3 RJ45SMD, T1 IRFR5305, T2 BC847BSMD, T3 BC847BSMD, X1 CSM-7X-DU

Commit message: add web
Parts:
- removed C4, C5: (no value), rcl:C-EUC0805
- removed R2: 10k, rcl:R-EU_R1206
- removed X1: CSM-7X-DU, crystal:CSM-7X-DU
- removed X2: (no value), sparkfun:CRYSTAL5X3
- added I2C_BUS1: RJ45SMD, con-tycoelectronics:RJ45SMD
Connections:
- net +12V: now also I2C_BUS1.1, I2C_BUS1.2; no longer C1.+
- net GND: now also I2C_BUS1.3, I2C_BUS1.4, I2C_BUS1.5; no longer C4.1, C5.1
- net IN: now also C1.+; no longer R2.2
- net LX: now also I2C_BUS1.8
- net LY: now also I2C_BUS1.6
- net N$26: no longer R2.1
- net N$49: no longer C4.2, X1.2, X2.2
- net N$50: no longer C5.2, X1.1, X2.1
- net VCC: now also I2C_BUS.7, I2C_BUS1.7
Other:
- moved on the sheet: C1, D1, R14, R15
