File: pcb/dimmer.v2.sch (EAGLE design)
At the start: 41 parts, among them M328 ATMEGA328P-AU, SW1 RJ45SMD, SW2 RJ45SMD, SW3 RJ45SMD, T1 IRFR5305, T2 BC847BSMD, T3 BC847BSMD

Commit message: initial add light
Parts:
- removed C2: 100nF, rcl:C-EUC1206
- removed D1: M1, diode:ES2D
- added C1: (no value), rcl:CPOL-EUC/6032-28W
- T1: value IRFR5305 -> IRFR024NPBF
Connections:
- removed net IN: C5.+, D1.C, L1117.IN
- net +12V: now also C5.+, L1117.IN; no longer D1.A
- net GND: now also C1.-; no longer C2.2
- net VCC: now also C1.+; no longer C2.1
Changed lines of the file:
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@@
 <?xml version="1.0" encoding="utf-8"?>
 <!DOCTYPE eagle SYSTEM "eagle.dtd">
-<eagle version="6.5.0">
+<eagle version="7.3.0">
 <drawing>
 <settings>
@@
 <layers>
 <layer number="1" name="Top" color="4" fill="1" visible="no" active="no"/>
+<layer number="2" name="Route2" color="1" fill="3" visible="no" active="no"/>
+<layer number="3" name="Route3" color="4" fill="3" visible="no" active="no"/>
+<layer number="4" name="Route4" color="1" fill="4" visible="no" active="no"/>
+<layer number="5" name="Route5" color="4" fill="4" visible="no" active="no"/>
+<layer number="6" name="Route6" color="1" fill="8" visible="no" active="no"/>
+<layer number="7" name="Route7" color="4" fill="8" visible="no" active="no"/>
+<layer number="8" name="Route8" color="1" fill="2" visible="no" active="no"/>
+<layer number="9" name="Route9" color="4" fill="2" visible="no" active="no"/>
+<layer number="10" name="Route10" color="1" fill="7" visible="no" active="no"/>
+<layer number="11" name="Route11" color="4" fill="7" visible="no" active="no"/>
+<layer number="12" name="Route12" color="1" fill="5" visible="no" active="no"/>
+<layer number="13" name="Route13" color="4" fill="5" visible="no" active="no"/>
+<layer number="14" name="Route14" color="1" fill="6" visible="no" active="no"/>
+<layer number="15" name="Route15" color="4" fill="6" visible="no" active="no"/>
 <layer number="16" name="Bottom" color="1" fill="1" visible="no" active="no"/>
 <layer number="17" name="Pads" color="2" fill="1" visible="no" active="no"/>
@@
 <parts>
 <part name="R6" library="rcl" deviceset="R-EU_" device="R1206" value="1K"/>
-<part name="T1" library="transistor-power" deviceset="IRF?5305" device="R"/>
+<part name="T1" library="transistor-power" deviceset="IRF?5305" device="R" value="IRFR024NPBF"/>
 <part name="AC-230V" library="con-wago-508" deviceset="W237-3E" device=""/>
 <part name="VCC+12V1" library="supply2" deviceset="VCC" device="" value="12V"/>
@@
 <part name="GND10" library="supply1" deviceset="GND" device=""/>
 <part name="+12V" library="supply2" deviceset="VCC" device=""/>
-<part name="C2" library="rcl" deviceset="C-EU" device="C1206" value="100nF"/>
 <part name="GND13" library="supply1" deviceset="GND" device=""/>
 <part name="C3" library="rcl" deviceset="C-EU" device="C1206" value="100nF"/>
@@
 <part name="T3" library="transistor-npn" deviceset="BC847*" device="SMD" technology="B"/>
 <part name="T2" library="transistor-npn" deviceset="BC847*" device="SMD" technology="B"/>
-<part name="D1" library="diode" deviceset="ES2D" device="" value="M1"/>
 <part name="GND4" library="supply1" deviceset="GND" device=""/>
 <part name="R8" library="rcl" deviceset="R-EU_" device="R1206" value="10k"/>
@@
 <part name="R16" library="rcl" deviceset="R-EU_" device="R1206" value="680"/>
 <part name="C5" library="rcl" deviceset="CPOL-EU" device="140CLH-0810" value="100uF"/>
+<part name="C1" library="rcl" deviceset="CPOL-EU" device="C/6032-28W"/>
 </parts>
 <sheets>
@@
 <instance part="GND10" gate="1" x="-97.79" y="199.39"/>
 <instance part="+12V" gate="G$1" x="-121.92" y="226.06" rot="R90"/>
-<instance part="C2" gate="G$1" x="-81.915" y="223.52" smashed="yes">
-<attribute name="NAME" x="-80.391" y="223.901" size="1.778" layer="95"/>
-<attribute name="VALUE" x="-80.391" y="218.821" size="1.778" layer="96"/>
-</instance>
 <instance part="GND13" gate="1" x="-81.915" y="215.9"/>
 <instance part="C3" gate="G$1" x="-48.895" y="213.36" smashed="yes" rot="R270">
@@
 <attribute name="VALUE" x="3.81" y="148.59" size="1.778" layer="96"/>
 </instance>
-<instance part="D1" gate="G$1" x="-115.57" y="226.06" smashed="yes">
-<attribute name="NAME" x="-118.11" y="228.1301" size="1.778" layer="95"/>
-<attribute name="VALUE" x="-118.11" y="222.1611" size="1.778" layer="96"/>
-</instance>
 <instance part="GND4" gate="1" x="-109.22" y="199.39"/>
 <instance part="R8" gate="G$1" x="62.23" y="212.09" rot="R90"/>
@@
 </instance>
 <instance part="C5" gate="G$1" x="-109.22" y="215.265"/>
+<instance part="C1" gate="G$1" x="-81.915" y="223.52"/>
 </instances>
 <busses>
@@
 <pinref part="GND9" gate="1" pin="GND"/>
 <wire x1="52.705" y1="217.17" x2="46.99" y2="217.17" width="0.1524" layer="91"/>
-</segment>
-<segment>
-<pinref part="C2" gate="G$1" pin="2"/>
-<pinref part="GND13" gate="1" pin="GND"/>
 </segment>
 <segment>
@@
 <wire x1="-109.22" y1="210.185" x2="-109.22" y2="201.93" width="0.1524" layer="91"/>
 </segment>
+<segment>
+<pinref part="GND13" gate="1" pin="GND"/>
+<pinref part="C1" gate="G$1" pin="-"/>
+</segment>
 </net>
 <net name="N$15" class="0">
@@
 <segment>
 <pinref part="+12V" gate="G$1" pin="VCC"/>
-<pinref part="D1" gate="G$1" pin="A"/>
-<wire x1="-118.11" y1="226.06" x2="-119.38" y2="226.06" width="0.1524" layer="91"/>
+<wire x1="-113.03" y1="226.06" x2="-119.38" y2="226.06" width="0.1524" layer="91"/>
 </segment>
 <segment>
@@
 <wire x1="-87.63" y1="233.045" x2="-84.455" y2="233.045" width="0.1524" layer="91"/>
 <junction x="-87.63" y="233.045"/>
+</segment>
+<segment>
+<pinref part="L1117" gate="G$1" pin="IN"/>
+<wire x1="-113.03" y1="226.06" x2="-109.22" y2="226.06" width="0.1524" layer="91"/>
+<pinref part="C5" gate="G$1" pin="+"/>
+<wire x1="-109.22" y1="226.06" x2="-105.41" y2="226.06" width="0.1524" layer="91"/>
+<wire x1="-109.22" y1="217.805" x2="-109.22" y2="226.06" width="0.1524" layer="91"/>
+<junction x="-109.22" y="226.06"/>
 </segment>
 </net>
@@
 <wire x1="-46.355" y1="226.06" x2="-70.485" y2="226.06" width="0.1524" layer="91"/>
 <wire x1="-70.485" y1="226.06" x2="-70.485" y2="220.345" width="0.1524" layer="91"/>
-<pinref part="C2" gate="G$1" pin="1"/>
-<wire x1="-81.915" y1="226.06" x2="-70.485" y2="226.06" width="0.1524" layer="91"/>
+<wire x1="-90.17" y1="226.06" x2="-81.915" y2="226.06" width="0.1524" layer="91"/>
 <junction x="-70.485" y="226.06"/>
 <pinref part="SUPPLY9" gate="G$1" pin="VCC"/>
 <junction x="-70.485" y="226.06"/>
 <pinref part="L1117" gate="G$1" pin="OUT"/>
-<wire x1="-90.17" y1="226.06" x2="-81.915" y2="226.06" width="0.1524" layer="91"/>
-<junction x="-81.915" y="226.06"/>
 <pinref part="M328" gate="A" pin="AVCC"/>
 <pinref part="R3" gate="G$1" pin="2"/>
+<pinref part="C1" gate="G$1" pin="+"/>
+<wire x1="-81.915" y1="226.06" x2="-70.485" y2="226.06" width="0.1524" layer="91"/>
+<junction x="-81.915" y="226.06"/>
 </segment>
 <segment>
@@
 </segment>
 </net>
-<net name="IN" class="0">
-<segment>
-<pinref part="D1" gate="G$1" pin="C"/>
-<pinref part="L1117" gate="G$1" pin="IN"/>
-<wire x1="-113.03" y1="226.06" x2="-109.22" y2="226.06" width="0.1524" layer="91"/>
-<pinref part="C5" gate="G$1" pin="+"/>
-<wire x1="-109.22" y1="226.06" x2="-105.41" y2="226.06" width="0.1524" layer="91"/>
-<wire x1="-109.22" y1="217.805" x2="-109.22" y2="226.06" width="0.1524" layer="91"/>
-<junction x="-109.22" y="226.06"/>
-</segment>
-</net>
 <net name="12V" class="0">
 <segment>
@@
 </sheet>
 </sheets>
-<errors>
-</errors>
 </schematic>
 </drawing>
