File: pcb/switch.m16.sch (EAGLE design)
At the start: 43 parts, among them IC1 MEGA16-A

Commit message: version 2.0
Parts:
- removed D1: BZX84CSMD, diode:BZX84CSMD
- removed N$39, TP1, TP10, TP12, TP14, TP2, TP3, TP4, TP5, TP6, TP7, TP9: TPSQTP15SQ, testpad:TPSQTP15SQ
- removed U$2: RJ45SMD, con-tycoelectronics:RJ45SMD
- removed U$6: MIMISMD, switch-misc:MIMISMD
- added C1, C2: (no value), rcl:C-EUC0805
- added INPUT: RJ45SMD, con-tycoelectronics:RJ45SMD
- added MEGA16A: MEGA16-A, avr-5:MEGA16-A
- added R13, R15: (no value), rcl:R-EU_R1206
- added R17, R18: 0, rcl:R-EU_R1206
- added TL1: MIMISMD, switch-misc:MIMISMD
- added Y1: (no value), sparkfun:CRYSTAL5X3
- C6, C7: value (none) -> 100nF
- IC1: value MEGA16-A -> (none); device avr-5:MEGA16-A -> sparkfun:V_REG_LM1117SOT223
- R1, R2, R3, R4, R5, R6, R7, R8: value (none) -> 1M
- R10, R9: value (none) -> 10k
- R11: value (none) -> 120
- R12, R16: value (none) -> 680
- R14: value (none) -> 0
- renumbered U$1 to I2C, U$3 to OUTPUT, U$4 to 485, U$5 to ISP
Connections:
- removed net N$14: IC1.(ADC0)PA0, R8.2, TP2.TP
- new net N$28: C1.2, MEGA16A.XTAL2, Y1.2
- new net N$29: C2.2, MEGA16A.XTAL1, Y1.1
- new net N$31: MEGA16A.(ADC4)PA4, R4.2
- new net N$35: MEGA16A.(ADC1)PA1, R7.2
- net +12V: now also INPUT.3, INPUT.4, R13.1, R13.2, R15.1, R15.2, R18.2; no longer R14.1, TP3.TP, TP4.TP, U$2.3, U$2.4
- net GND: now also C1.1, C2.1, INPUT.1, INPUT.2, MEGA16A.GND, MEGA16A.GND1, MEGA16A.GND2, R14.1, TL1.S, TL1.S@1; no longer D1.A, IC1.GND, IC1.GND1, IC1.GND2, U$2.1, U$2.2
- net N$1: now also MEGA16A.(OC1B)PD4; no longer IC1.(OC1B)PD4
- net N$10: now also MEGA16A.PC0(SCL); no longer IC1.PC0(SCL)
- net N$11: now also MEGA16A.PC1(SDA); no longer IC1.PC1(SDA)
- net N$12: now also INPUT.7; no longer U$2.7
- net N$13: now also INPUT.8; no longer U$2.8
- net N$15: now also MEGA16A.(RXD)PD0; no longer IC1.(RXD)PD0
- net N$16: now also MEGA16A.(TXD)PD1; no longer IC1.(TXD)PD1
- net N$17: now also MEGA16A.(INT0)PD2; no longer IC1.(INT0)PD2
- net N$18: now also MEGA16A.(INT1)PD3; no longer IC1.(INT1)PD3
- net N$19: now also MEGA16A.(MISO)PB6; no longer IC1.(MISO)PB6
- net N$2: now also MEGA16A.(SS)PB4; no longer IC1.(SS)PB4
- net N$20: now also MEGA16A.(SCK)PB7; no longer IC1.(SCK)PB7
- net N$21: now also MEGA16A.RESET; no longer IC1.RESET
- net N$22: now also MEGA16A.(MOSI)PB5; no longer IC1.(MOSI)PB5
- net N$3: now also IC1.ADJ, R14.2, R17.2; no longer IC1.(ADC7)PA7, R1.2, TP7.TP
- net N$32: now also MEGA16A.(TDO)PC4, R10.1, TL1.P, TL1.P@1; no longer IC1.(TDO)PC4, U$6.P, U$6.P@1
- net N$34: now also MEGA16A.(ADC5)PA5, R3.2; no longer R10.1, U$6.S, U$6.S@1
- net N$36: now also MEGA16A.AREF; no longer IC1.AREF
- net N$4: now also MEGA16A.(ADC6)PA6; no longer IC1.(ADC6)PA6, TP9.TP
- net N$5: now also MEGA16A.(ADC7)PA7, R1.2; no longer IC1.(ADC5)PA5, R3.2, TP12.TP
- net N$6: now also MEGA16A.(ADC0)PA0, R8.2; no longer IC1.(ADC4)PA4, R4.2, TP14.TP
- net N$7: now also MEGA16A.(ADC3)PA3; no longer IC1.(ADC3)PA3, N$39.TP
- net N$8: now also MEGA16A.(ADC2)PA2; no longer IC1.(ADC2)PA2, TP10.TP
- net N$9: now also IC1.IN, R18.1; no longer IC1.(ADC1)PA1, R7.2, TP1.TP
- net VCC: now also IC1.OUT, INPUT.5, INPUT.6, MEGA16A.AVCC, MEGA16A.VCC, R17.1; no longer D1.C, IC1.AVCC, IC1.VCC, R14.2, TP5.TP, TP6.TP, U$2.5, U$2.6
Other:
- moved on the sheet: C5, C6, C7, LED1, R10, R14, R16

Commit message: sens
Parts:
- removed C5: (no value), rcl:C-EUC1206
- removed I2C: P82B715, i2c:P82B715
- removed INPUT: RJ45SMD, con-tycoelectronics:RJ45SMD
- removed R15: (no value), rcl:R-EU_R1206
- removed R17, R18: 0, rcl:R-EU_R1206
- removed TL1: MIMISMD, switch-misc:MIMISMD
- added C3: (no value), rcl:CPOL-EUSMCC
- added D1: ES2D, diode:ES2D
- added TEMP_SENZ: TCN75, linear:TCN75
- R10: value 10k -> 4k7
- R13: value (none) -> 4k7
- R14: value 0 -> 10k
- renumbered OUTPUT to DIMMER_UTP
Connections:
- removed net N$13: I2C.LCL, INPUT.8
- removed net N$32: MEGA16A.(TDO)PC4, R10.1, TL1.P, TL1.P@1
- removed net N$9: IC1.IN, R18.1
- net +12V: now also D1.A; no longer I2C.VCC, INPUT.3, INPUT.4, R13.1, R13.2, R15.1, R15.2, R18.2
- net GND: now also C3.-, IC1.ADJ, R14.2, TEMP_SENZ.A0, TEMP_SENZ.A1, TEMP_SENZ.A2, TEMP_SENZ.GND; no longer C5.2, I2C.GND, INPUT.1, INPUT.2, TL1.S, TL1.S@1
- net N$10: now also R13.2, TEMP_SENZ.SCL; no longer I2C.SCL
- net N$11: now also R10.2, TEMP_SENZ.SDA; no longer I2C.SDA
- net N$12: now also MEGA16A.(TCK)PC2, TEMP_SENZ.ALERT; no longer I2C.LDA, INPUT.7
- net N$3: now also C3.+, D1.C, IC1.IN; no longer IC1.ADJ, R14.2, R17.2
- net VCC: now also R10.1, R13.1, TEMP_SENZ.VCC; no longer C5.1, INPUT.5, INPUT.6, R10.2, R17.1
Other:
- moved on the sheet: IC1, R10, R13, R14

Commit message: initial add light
Parts:
- added LED7: (no value), led:LEDSML1206
- added R15: 4k7, rcl:R-EU_R1206
- R14: value 10k -> 0
Connections:
- new net N$13: LED7.A, R15.2
- new net N$9: MEGA16A.(TOSC1)PC6, R15.1
- new net PC5: MEGA16A.(TDI)PC5
- net GND: now also LED7.C
Other:
- moved on the sheet: R10, R13, R16
Changed lines of the file:
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@@
 <setting verticaltext="up"/>
 </settings>
-<grid distance="0.025" unitdist="inch" unit="inch" style="lines" multiple="1" display="no" altdistance="0.01" altunitdist="inch" altunit="inch"/>
+<grid distance="0.1" unitdist="inch" unit="inch" style="lines" multiple="1" display="no" altdistance="0.01" altunitdist="inch" altunit="inch"/>
 <layers>
 <layer number="1" name="Top" color="4" fill="1" visible="no" active="no"/>
@@
 <part name="D1" library="diode" deviceset="ES2D" device=""/>
 <part name="C3" library="rcl" deviceset="CPOL-EU" device="SMCC"/>
-<part name="R14" library="rcl" deviceset="R-EU_" device="R1206" value="10k"/>
+<part name="R14" library="rcl" deviceset="R-EU_" device="R1206" value="0"/>
+<part name="R15" library="rcl" deviceset="R-EU_" device="R1206" value="4k7"/>
+<part name="LED7" library="led" deviceset="LED" device="SML1206"/>
+<part name="GND15" library="supply1" deviceset="GND" device=""/>
 </parts>
 <sheets>
@@
 <instance part="+12V" gate="G$1" x="-74.295" y="81.28" rot="R90"/>
 <instance part="GND13" gate="1" x="-58.42" y="59.055"/>
-<instance part="R16" gate="G$1" x="60.325" y="48.26"/>
+<instance part="R16" gate="G$1" x="57.785" y="48.26"/>
 <instance part="LED1" gate="G$1" x="46.99" y="48.26" rot="R90"/>
-<instance part="GND16" gate="1" x="65.405" y="45.085"/>
+<instance part="GND16" gate="1" x="62.865" y="45.085"/>
 <instance part="LED3" gate="G$1" x="59.69" y="16.51" rot="R90"/>
 <instance part="LED4" gate="G$1" x="51.435" y="16.51" rot="R90"/>
@@
 <instance part="GND14" gate="1" x="105.41" y="22.86"/>
 <instance part="GND9" gate="1" x="80.01" y="22.86"/>
-<instance part="R10" gate="G$1" x="52.07" y="35.56" rot="R270"/>
-<instance part="R13" gate="G$1" x="58.42" y="35.56" rot="R270"/>
-<instance part="SUPPLY7" gate="G$1" x="46.355" y="40.64" rot="R90"/>
+<instance part="R10" gate="G$1" x="69.215" y="35.56" smashed="yes" rot="R270">
+<attribute name="NAME" x="71.9836" y="37.465" size="1.778" layer="95" rot="R270"/>
+<attribute name="VALUE" x="66.548" y="32.385" size="1.778" layer="96" rot="R270"/>
+</instance>
+<instance part="R13" gate="G$1" x="64.135" y="35.56" smashed="yes" rot="R270">
+<attribute name="NAME" x="65.6336" y="37.465" size="1.778" layer="95" rot="R270"/>
+<attribute name="VALUE" x="61.468" y="32.385" size="1.778" layer="96" rot="R270"/>
+</instance>
+<instance part="SUPPLY7" gate="G$1" x="69.215" y="43.815"/>
 <instance part="GND6" gate="1" x="-66.675" y="59.055"/>
 <instance part="GND11" gate="1" x="-66.675" y="74.93" rot="R180"/>
@@
 <instance part="C3" gate="G$1" x="-58.42" y="70.485"/>
 <instance part="R14" gate="G$1" x="-66.675" y="66.675" rot="R90"/>
+<instance part="R15" gate="G$1" x="45.085" y="38.1"/>
+<instance part="LED7" gate="G$1" x="52.705" y="38.1" rot="R90"/>
+<instance part="GND15" gate="1" x="57.785" y="35.56"/>
 </instances>
 <busses>
@@
 <pinref part="R16" gate="G$1" pin="2"/>
 <pinref part="GND16" gate="1" pin="GND"/>
-<wire x1="65.405" y1="48.26" x2="65.405" y2="47.625" width="0.1524" layer="91"/>
+<wire x1="62.865" y1="48.26" x2="62.865" y2="47.625" width="0.1524" layer="91"/>
 </segment>
 <segment>
@@
 <pinref part="R14" gate="G$1" pin="1"/>
 </segment>
+<segment>
+<pinref part="LED7" gate="G$1" pin="C"/>
+<pinref part="GND15" gate="1" pin="GND"/>
+</segment>
 </net>
 <net name="+12V" class="0">
@@
 <pinref part="LED1" gate="G$1" pin="C"/>
 <pinref part="R16" gate="G$1" pin="1"/>
-<wire x1="55.245" y1="48.26" x2="52.07" y2="48.26" width="0.1524" layer="91"/>
+<wire x1="52.705" y1="48.26" x2="52.07" y2="48.26" width="0.1524" layer="91"/>
 </segment>
 </net>
@@
 <segment>
 <pinref part="MEGA16A" gate="G$1" pin="PC0(SCL)"/>
-<wire x1="37.465" y1="22.86" x2="58.42" y2="22.86" width="0.1524" layer="91"/>
-<wire x1="58.42" y1="22.86" x2="74.295" y2="22.86" width="0.1524" layer="91"/>
+<wire x1="37.465" y1="22.86" x2="64.135" y2="22.86" width="0.1524" layer="91"/>
+<wire x1="64.135" y1="22.86" x2="74.295" y2="22.86" width="0.1524" layer="91"/>
 <wire x1="74.295" y1="22.86" x2="74.295" y2="40.64" width="0.1524" layer="91"/>
 <wire x1="74.295" y1="40.64" x2="80.01" y2="40.64" width="0.1524" layer="91"/>
 <pinref part="TEMP_SENZ" gate="G$1" pin="SCL"/>
 <pinref part="R13" gate="G$1" pin="2"/>
-<wire x1="58.42" y1="30.48" x2="58.42" y2="22.86" width="0.1524" layer="91"/>
-<junction x="58.42" y="22.86"/>
+<wire x1="64.135" y1="30.48" x2="64.135" y2="22.86" width="0.1524" layer="91"/>
+<junction x="64.135" y="22.86"/>
 </segment>
 </net>
@@
 <wire x1="71.755" y1="45.72" x2="71.755" y2="25.4" width="0.1524" layer="91"/>
 <pinref part="MEGA16A" gate="G$1" pin="PC1(SDA)"/>
-<wire x1="71.755" y1="25.4" x2="52.07" y2="25.4" width="0.1524" layer="91"/>
-<wire x1="52.07" y1="25.4" x2="37.465" y2="25.4" width="0.1524" layer="91"/>
+<wire x1="71.755" y1="25.4" x2="69.215" y2="25.4" width="0.1524" layer="91"/>
+<wire x1="69.215" y1="25.4" x2="37.465" y2="25.4" width="0.1524" layer="91"/>
 <wire x1="71.755" y1="45.72" x2="80.01" y2="45.72" width="0.1524" layer="91"/>
 <pinref part="TEMP_SENZ" gate="G$1" pin="SDA"/>
 <pinref part="R10" gate="G$1" pin="2"/>
-<wire x1="52.07" y1="30.48" x2="52.07" y2="25.4" width="0.1524" layer="91"/>
-<junction x="52.07" y="25.4"/>
+<wire x1="69.215" y1="30.48" x2="69.215" y2="25.4" width="0.1524" layer="91"/>
+<junction x="69.215" y="25.4"/>
 </segment>
 </net>
@@
 <pinref part="SUPPLY7" gate="G$1" pin="VCC"/>
 <pinref part="R10" gate="G$1" pin="1"/>
-<wire x1="48.895" y1="40.64" x2="52.07" y2="40.64" width="0.1524" layer="91"/>
+<wire x1="69.215" y1="41.275" x2="69.215" y2="40.64" width="0.1524" layer="91"/>
 <pinref part="R13" gate="G$1" pin="1"/>
-<wire x1="58.42" y1="40.64" x2="52.07" y2="40.64" width="0.1524" layer="91"/>
-<junction x="52.07" y="40.64"/>
+<wire x1="64.135" y1="40.64" x2="69.215" y2="40.64" width="0.1524" layer="91"/>
+<junction x="69.215" y="40.64"/>
 </segment>
 </net>
@@
 </segment>
 </net>
+<net name="N$9" class="0">
+<segment>
+<pinref part="MEGA16A" gate="G$1" pin="(TOSC1)PC6"/>
+<pinref part="R15" gate="G$1" pin="1"/>
+<wire x1="40.005" y1="38.1" x2="37.465" y2="38.1" width="0.1524" layer="91"/>
+</segment>
+</net>
+<net name="N$13" class="0">
+<segment>
+<pinref part="R15" gate="G$1" pin="2"/>
+<pinref part="LED7" gate="G$1" pin="A"/>
+</segment>
+</net>
+<net name="PC5" class="0">
+<segment>
+<pinref part="MEGA16A" gate="G$1" pin="(TDI)PC5"/>
+<wire x1="37.465" y1="35.56" x2="40.005" y2="35.56" width="0.1524" layer="91"/>
+</segment>
+</net>
