File: pcb/dimmer.light.sch (EAGLE design)
At the start: 21 parts, among them IC1 NCP1117ST50T3G, SW1 RJ45SMD, T1 IRFR024NPBF, T2 BC847BSMD, U1 ATTINY2313

Commit message: final version
Parts:
- R4: value 120 -> 220
Changed lines of the file:
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@@
 <setting verticaltext="up"/>
 </settings>
-<grid distance="25" unitdist="mil" unit="mil" style="lines" multiple="1" display="no" altdistance="0.01" altunitdist="inch" altunit="inch"/>
+<grid distance="0.1" unitdist="inch" unit="inch" style="lines" multiple="1" display="no" altdistance="0.01" altunitdist="inch" altunit="inch"/>
 <layers>
 <layer number="1" name="Top" color="4" fill="1" visible="no" active="no"/>
@@
 <part name="GND6" library="supply1" deviceset="GND" device=""/>
 <part name="GND14" library="supply1" deviceset="GND" device=""/>
-<part name="R4" library="rcl" deviceset="R-EU_" device="R1206" value="120"/>
+<part name="R4" library="rcl" deviceset="R-EU_" device="R1206" value="220"/>
 <part name="LED1" library="led" deviceset="LED" device="SML1206"/>
 <part name="R5" library="rcl" deviceset="R-EU_" device="R1206" value="680"/>
