File: pcb/switch.m16.brd (EAGLE design)
At the start: 78.1 x 77.8 mm, 43 parts, among them IC1 MEGA16-A

Commit message: version 2.0
Parts:
- removed D1: BZX84CSMD, diode:TO236
- removed N$39, TP1, TP10, TP12, TP14, TP2, TP3, TP4, TP5, TP6, TP7, TP9: TPSQTP15SQ, testpad:TP15SQ
- removed U$2, U$3: RJ45SMD, con-tycoelectronics:RJ45SMD
- removed U$4: MAX485SMD, maxim:SO08
- removed U$6: MIMISMD, switch-misc:MINISMD
- added 485: MAX485SMD, maxim:SO08
- added C1, C2: (no value), rcl:C0805
- added INPUT, OUTPUT: RJ45SMD, con-tycoelectronics:RJ45SMD
- added MEGA16A: MEGA16-A, avr-5:TQFP44
- added R13, R15: (no value), rcl:R1206
- added R17, R18: 0, rcl:R1206
- added TL1: MIMISMD, switch-misc:MINISMD
- added Y1: (no value), sparkfun:CRYSTAL-SMD-5X3
- C6, C7: value (none) -> 100nF
- IC1: value MEGA16-A -> (none); device avr-5:TQFP44 -> sparkfun:SOT223
- R1, R2, R3, R4, R5, R6, R7, R8: value (none) -> 1M
- R10, R9: value (none) -> 10k
- R11: value (none) -> 120
- R12, R16: value (none) -> 680
- R14: value (none) -> 0
- moved IC1 30.7 mm to (24.0, 66.2), turned to 0 degrees
- moved R14 12.5 mm to (17.3, 64.3), turned to 0 degrees
- moved R9 9.22 mm to (28.1, 15.4)
- moved LED2 4.97 mm to (37.9, 22.1), turned to 90 degrees
- moved R11 4.45 mm to (42.1, 11.9)
- moved C6 3.49 mm to (17.3, 60.5)
- moved C5 2.86 mm to (17.3, 57.3)
- moved R16 2.70 mm to (15.1, 35.7)
- moved C7 2.54 mm to (17.3, 54.3)
- moved LED1 2.36 mm to (18.1, 35.4)
- moved LED5 2.06 mm to (35.6, 1.75)
- moved R8 1.81 mm to (14.3, 12.5)
- moved LED3 1.59 mm to (35.2, 70.8)
- moved R10 0.97 mm to (30.2, 63.8), turned to 90 degrees
- moved R1 0.64 mm to (17.3, 51.3)
- renumbered U$1 to I2C, U$5 to ISP
Connections:
- removed net N$14: IC1.37, R8.2, TP2.TP
- new net N$28: C1.2, MEGA16A.7, Y1.3
- new net N$29: C2.2, MEGA16A.8, Y1.1
- new net N$31: MEGA16A.33, R4.2
- new net N$35: MEGA16A.36, R7.2
- net +12V: now also INPUT.P$3, INPUT.P$4, OUTPUT.P$3, OUTPUT.P$4, R13.1, R13.2, R15.1, R15.2, R18.2; no longer R14.1, TP3.TP, TP4.TP, U$2.P$3, U$2.P$4, U$3.P$3, U$3.P$4
- net AGND: now also MEGA16A.28; no longer IC1.28
- net GND: now also 485.5, C1.1, C2.1, INPUT.P$1, INPUT.P$2, MEGA16A.18, MEGA16A.39, MEGA16A.6, OUTPUT.P$1, OUTPUT.P$2, R14.1, TL1.P$2, TL1.P$4; no longer D1.A, IC1.18, IC1.39, IC1.6, U$2.P$1, U$2.P$2, U$3.P$1, U$3.P$2, U$4.5
- net N$1: now also MEGA16A.13; no longer IC1.13
- net N$10: now also MEGA16A.19; no longer IC1.19
- net N$11: now also MEGA16A.20; no longer IC1.20
- net N$12: now also INPUT.P$7; no longer U$2.P$7
- net N$13: now also INPUT.P$8; no longer U$2.P$8
- net N$15: now also 485.1, MEGA16A.9; no longer IC1.9, U$4.1
- net N$16: now also 485.4, MEGA16A.10; no longer IC1.10, U$4.4
- net N$17: now also 485.2, 485.3, MEGA16A.11; no longer IC1.11, U$4.2, U$4.3
- net N$18: now also MEGA16A.12; no longer IC1.12
- net N$19: now also MEGA16A.2; no longer IC1.2
- net N$2: now also MEGA16A.44; no longer IC1.44
- net N$20: now also MEGA16A.3; no longer IC1.3
- net N$21: now also MEGA16A.4; no longer IC1.4
- net N$22: now also MEGA16A.1; no longer IC1.1
- net N$23: now also 485.6, OUTPUT.P$7; no longer U$3.P$7, U$4.6
- net N$24: now also 485.7, OUTPUT.P$8; no longer U$3.P$8, U$4.7
- net N$3: now also IC1.1, R14.2, R17.2; no longer IC1.30, R1.2, TP7.TP
- net N$32: now also MEGA16A.23, R10.1, TL1.P$1, TL1.P$3; no longer IC1.23, U$6.P$1, U$6.P$3
- net N$34: now also MEGA16A.32, R3.2; no longer R10.1, U$6.P$2, U$6.P$4
- net N$36: now also MEGA16A.29; no longer IC1.29
- net N$4: now also MEGA16A.31; no longer IC1.31, TP9.TP
- net N$5: now also MEGA16A.30, R1.2; no longer IC1.32, R3.2, TP12.TP
- net N$6: now also MEGA16A.37, R8.2; no longer IC1.33, R4.2, TP14.TP
- net N$7: now also MEGA16A.34; no longer IC1.34, N$39.TP
- net N$8: now also MEGA16A.35; no longer IC1.35, TP10.TP
- net N$9: now also IC1.3, R18.1; no longer IC1.36, R7.2, TP1.TP
- net VCC: now also 485.8, IC1.2, INPUT.P$5, INPUT.P$6, MEGA16A.27, MEGA16A.5, OUTPUT.P$5, OUTPUT.P$6, R17.1; no longer D1.C, IC1.27, IC1.5, R14.2, TP5.TP, TP6.TP, U$2.P$5, U$2.P$6, U$3.P$5, U$3.P$6, U$4.8
- net VCC1: now also MEGA16A.17; no longer IC1.17
- net VCC2: now also MEGA16A.38; no longer IC1.38
Routing:
- net GND: track 413.4 -> 316.8 mm
- net +12V: track 149.0 -> 102.5 mm
- net N$35: track 0.00 -> 46.4 mm, vias 0 -> 1
- net N$21: track 29.7 -> 64.3 mm
- net N$9: track 42.6 -> 8.41 mm
- net VCC: track 208.4 -> 179.4 mm
- net N$14: track 32.8 -> 5.71 mm
- net N$29: track 0.00 -> 21.0 mm
- net N$34: track 8.90 -> 29.7 mm, vias 0 -> 1
- net N$31: track 0.00 -> 20.4 mm, vias 0 -> 1
- net N$20: track 23.9 -> 40.0 mm
- net N$19: track 16.1 -> 31.2 mm
- net N$32: track 25.6 -> 40.6 mm
- net N$6: track 21.6 -> 35.9 mm, vias 0 -> 2
- net N$28: track 0.00 -> 13.0 mm
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- added copper zone on layer 16, net N$31
- added copper zone on layer 16, net N$34
- added copper zone on layer 16, net N$35
- added copper zone on layer 16, net N$44
- added copper zone on layer 16, net N$5
- added copper zone on layer 16, net N$6
- added copper zone on layer 16, net N$7
- added copper zone on layer 16, net N$8
- removed copper zone on layer 16, net N$25
- removed copper zone on layer 16, net N$26
- removed copper zone on layer 16, net N$27
- removed copper zone on layer 16, net N$28
- removed copper zone on layer 16, net N$29
- removed copper zone on layer 16, net N$39
- removed copper zone on layer 16, net N$40
- removed copper zone on layer 16, net N$42
Other:
- board size 78.1 x 77.8 mm -> 77.8 x 77.8 mm
- board text added: "+5V"
- board text added: "12V"
- board text added: "5V"
- board text added: "A"
- board text added: "B"
- board text added: "GND"
- board text added: "IN"
- board text added: "LCL"
- board text added: "LDA"
- board text added: "MISO"
- board text added: "MOSI"
- board text added: "OUT"
- board text added: "PC2"
- board text added: "PC3"
- board text added: "PC5"
- board text added: "RST"
- board text added: "RX"
- board text added: "S1"
- board text added: "SCK"
- board text added: "SCL"
- board text added: "SDA"
- board text added: "TX"

Commit message: sens
Parts:
- removed C5: (no value), rcl:C1206
- removed I2C: P82B715, i2c:P82B715SMD
- removed INPUT, OUTPUT: RJ45SMD, con-tycoelectronics:RJ45SMD
- removed R15: (no value), rcl:R1206
- removed R17, R18: 0, rcl:R1206
- removed TL1: MIMISMD, switch-misc:MINISMD
- added C3: (no value), rcl:SMC_C
- added D1: ES2D, diode:SMB
- added DIMMER_UTP: RJ45SMD, con-tycoelectronics:RJ45SMD
- added TEMP_SENZ: TCN75, linear:SO08
- R10: value 10k -> 4k7
- R13: value (none) -> 4k7
- R14: value 0 -> 10k
- moved R14 31.9 mm to (47.5, 53.8), turned to 90 degrees
- moved R10 23.0 mm to (44.9, 46.2), turned to 0 degrees
- moved R13 19.8 mm to (39.2, 47.5), turned to 270 degrees
- moved IC1 16.7 mm to (40.0, 61.4), turned to 90 degrees
- moved C1 3.81 mm to (23.5, 27.3), turned to 0 degrees
- moved R11 3.24 mm to (42.7, 15.1)
- moved R16 2.73 mm to (16.7, 37.9)
- moved LED1 2.56 mm to (19.4, 37.6)
- moved MEGA16A 2.22 mm to (28.7, 39.2)
- moved R1 1.91 mm to (17.3, 53.2)
- moved R12 1.75 mm to (36.5, 27.6)
- moved C7 1.59 mm to (17.3, 55.9)
- moved C6 1.59 mm to (17.3, 58.9)
- moved C2 1.27 mm to (22.5, 23.5)
- moved Y1 1.11 mm to (27.9, 24.4)
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Connections:
- removed net N$13: I2C.2, INPUT.P$8
- removed net N$32: MEGA16A.23, R10.1, TL1.P$1, TL1.P$3
- removed net N$9: IC1.3, R18.1
- net +12V: now also D1.A, DIMMER_UTP.P$3, DIMMER_UTP.P$4; no longer I2C.8, INPUT.P$3, INPUT.P$4, OUTPUT.P$3, OUTPUT.P$4, R13.1, R13.2, R15.1, R15.2, R18.2
- net GND: now also C3.-, DIMMER_UTP.P$1, DIMMER_UTP.P$2, IC1.1, R14.2, TEMP_SENZ.4, TEMP_SENZ.5, TEMP_SENZ.6, TEMP_SENZ.7; no longer C5.2, I2C.4, INPUT.P$1, INPUT.P$2, OUTPUT.P$1, OUTPUT.P$2, TL1.P$2, TL1.P$4
- net N$10: now also R13.2, TEMP_SENZ.2; no longer I2C.3
- net N$11: now also R10.2, TEMP_SENZ.1; no longer I2C.6
- net N$12: now also MEGA16A.21, TEMP_SENZ.3; no longer I2C.7, INPUT.P$7
- net N$23: now also DIMMER_UTP.P$7; no longer OUTPUT.P$7
- net N$24: now also DIMMER_UTP.P$8; no longer OUTPUT.P$8
- net N$3: now also C3.+, D1.C, IC1.3; no longer IC1.1, R14.2, R17.2
- net VCC: now also DIMMER_UTP.P$5, DIMMER_UTP.P$6, R10.1, R13.1, TEMP_SENZ.8; no longer C5.1, INPUT.P$5, INPUT.P$6, OUTPUT.P$5, OUTPUT.P$6, R10.2, R17.1
Routing:
- net GND: track 316.8 -> 175.8 mm
- net +12V: track 102.5 -> 5.72 mm
- net N$3: track 12.1 -> 106.0 mm
- net N$32: track 40.6 -> 0.00 mm
- net N$10: track 15.9 -> 43.1 mm
- net N$13: track 24.9 -> 0.00 mm
- net N$12: track 22.5 -> 34.2 mm
- net N$11: track 12.7 -> 24.4 mm
- net N$25: track 10.3 -> 0.00 mm
- net N$9: track 8.41 -> 0.00 mm
- net N$18: track 87.8 -> 94.1 mm
- net N$24: track 32.1 -> 36.6 mm
- net VCC: track 179.4 -> 183.3 mm
- net N$23: track 42.6 -> 46.2 mm
- net N$5: track 20.4 -> 23.6 mm, vias 2 -> 1
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Other:
- board size 77.8 x 77.8 mm -> 78.9 x 77.8 mm
- board text removed: "LCL"
- board text removed: "LDA"
- board text removed: "PC2"

Commit message: initial add light
Parts:
- added LED7: (no value), led:SML1206
- added R15: 4k7, rcl:R1206
- R14: value 10k -> 0
- moved R14 4.45 mm to (50.3, 57.2)
- moved LED3 3.16 mm to (38.1, 72.2)
- moved 485 3.16 mm to (36.7, 18.0)
- moved C3 3.16 mm to (55.1, 63.4)
- moved LED1 3.16 mm to (22.2, 39.0)
- moved LED2 3.16 mm to (40.8, 22.8)
- moved R16 3.16 mm to (19.5, 39.3)
- moved R9 3.16 mm to (31.0, 16.7)
- moved TEMP_SENZ 3.16 mm to (59.1, 42.9)
- moved LED6 3.16 mm to (3.81, 38.0)
- moved ISP 3.16 mm to (22.5, 14.7)
- moved R11 3.16 mm to (45.6, 16.4)
- moved R3 3.16 mm to (9.84, 55.6)
- moved R4 3.16 mm to (9.84, 45.0)
- moved R8 3.16 mm to (17.1, 13.9)
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Connections:
- new net N$13: LED7.A, R15.2
- new net N$9: MEGA16A.25, R15.1
- new net PC5: MEGA16A.24
- net GND: now also LED7.C
Routing:
- net N$6: track 36.9 -> 59.6 mm
- net N$5: track 23.6 -> 44.7 mm
- net N$9: track 0.00 -> 14.8 mm
- net GND: track 175.8 -> 187.4 mm
- net N$26: track 7.88 -> 0.00 mm
- net N$10: track 43.1 -> 35.5 mm
- net N$44: track 1.11 -> 7.54 mm
- net N$14: track 5.72 -> 0.00 mm
- net PC5: track 0.00 -> 5.33 mm
- net N$4: track 40.2 -> 37.3 mm
- net N$31: track 20.4 -> 22.9 mm
- net N$8: track 37.4 -> 39.6 mm
- net N$3: track 106.0 -> 103.8 mm
- net VCC: track 183.3 -> 185.4 mm
- net N$13: track 0.00 -> 1.75 mm
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Other:
- board size 78.9 x 77.8 mm -> 75.1 x 75.2 mm
- board text removed: "PC3"
